File: ProstheticsEagle/circuitdraft.sch (EAGLE design)
At the start: 49 parts, among them IC1 BQ25887RGER, IC2 TPS54627DDAR, Q1 16 MHz

Commit message: ffff
Parts:
- L2: device rcl:L-US0204/7 -> SamacSys_Parts:TFM201610GHM-1R0MTAA
- renumbered SERVO1 to S1, SERVO2 to S2, SERVO3 to S3, SERVO4 to S4, SERVO5 to S5
Changed lines of the file:
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@@
 <parts>
 <part name="FRAME1" library="frames" library_urn="urn:adsk.eagle:library:229" deviceset="A3L-LOC" device=""/>
-<part name="SERVO1" library="pinhead" library_urn="urn:adsk.eagle:library:325" deviceset="PINHD-1X3" device="" package3d_urn="urn:adsk.eagle:package:22458/2"/>
-<part name="SERVO2" library="pinhead" library_urn="urn:adsk.eagle:library:325" deviceset="PINHD-1X3" device="" package3d_urn="urn:adsk.eagle:package:22458/2"/>
-<part name="SERVO3" library="pinhead" library_urn="urn:adsk.eagle:library:325" deviceset="PINHD-1X3" device="" package3d_urn="urn:adsk.eagle:package:22458/2"/>
-<part name="SERVO4" library="pinhead" library_urn="urn:adsk.eagle:library:325" deviceset="PINHD-1X3" device="" package3d_urn="urn:adsk.eagle:package:22458/2"/>
-<part name="SERVO5" library="pinhead" library_urn="urn:adsk.eagle:library:325" deviceset="PINHD-1X3" device="" package3d_urn="urn:adsk.eagle:package:22458/2"/>
+<part name="S1" library="pinhead" library_urn="urn:adsk.eagle:library:325" deviceset="PINHD-1X3" device="" package3d_urn="urn:adsk.eagle:package:22458/2"/>
+<part name="S2" library="pinhead" library_urn="urn:adsk.eagle:library:325" deviceset="PINHD-1X3" device="" package3d_urn="urn:adsk.eagle:package:22458/2"/>
+<part name="S3" library="pinhead" library_urn="urn:adsk.eagle:library:325" deviceset="PINHD-1X3" device="" package3d_urn="urn:adsk.eagle:package:22458/2"/>
+<part name="S4" library="pinhead" library_urn="urn:adsk.eagle:library:325" deviceset="PINHD-1X3" device="" package3d_urn="urn:adsk.eagle:package:22458/2"/>
+<part name="S5" library="pinhead" library_urn="urn:adsk.eagle:library:325" deviceset="PINHD-1X3" device="" package3d_urn="urn:adsk.eagle:package:22458/2"/>
 <part name="MYO" library="pinhead" library_urn="urn:adsk.eagle:library:325" deviceset="PINHD-1X3" device="" package3d_urn="urn:adsk.eagle:package:22458/2"/>
 <part name="AGND7" library="supply1" library_urn="urn:adsk.eagle:library:371" deviceset="AGND" device=""/>
@@
 <part name="C15" library="rcl" library_urn="urn:adsk.eagle:library:334" deviceset="C-US" device="C0805" package3d_urn="urn:adsk.eagle:package:23617/2" value="47 nF"/>
 <part name="AGND20" library="supply1" library_urn="urn:adsk.eagle:library:371" deviceset="AGND" device=""/>
-<part name="L2" library="rcl" library_urn="urn:adsk.eagle:library:334" deviceset="L-US" device="0204/7" package3d_urn="urn:adsk.eagle:package:23498/2" value="1 uH"/>
+<part name="L2" library="SamacSys_Parts" deviceset="TFM201610GHM-1R0MTAA" device="" value="1 uH"/>
 <part name="C16" library="rcl" library_urn="urn:adsk.eagle:library:334" deviceset="C-US" device="C0805" package3d_urn="urn:adsk.eagle:package:23617/2" value="44 uF"/>
 <part name="AGND21" library="supply1" library_urn="urn:adsk.eagle:library:371" deviceset="AGND" device=""/>
@@
 <attribute name="SHEET" x="357.505" y="5.08" size="2.54" layer="94"/>
 </instance>
-<instance part="SERVO1" gate="A" x="144.78" y="215.9" smashed="yes" rot="R270">
+<instance part="S1" gate="A" x="144.78" y="215.9" smashed="yes" rot="R270">
 <attribute name="NAME" x="150.495" y="222.25" size="1.778" layer="95" rot="R270"/>
 <attribute name="VALUE" x="137.16" y="222.25" size="1.778" layer="96" rot="R270"/>
 </instance>
-<instance part="SERVO2" gate="A" x="162.56" y="215.9" smashed="yes" rot="R270">
+<instance part="S2" gate="A" x="162.56" y="215.9" smashed="yes" rot="R270">
 <attribute name="NAME" x="168.275" y="222.25" size="1.778" layer="95" rot="R270"/>
 <attribute name="VALUE" x="154.94" y="222.25" size="1.778" layer="96" rot="R270"/>
 </instance>
-<instance part="SERVO3" gate="A" x="182.88" y="215.9" smashed="yes" rot="R270">
+<instance part="S3" gate="A" x="182.88" y="215.9" smashed="yes" rot="R270">
 <attribute name="NAME" x="188.595" y="222.25" size="1.778" layer="95" rot="R270"/>
 <attribute name="VALUE" x="175.26" y="222.25" size="1.778" layer="96" rot="R270"/>
 </instance>
-<instance part="SERVO4" gate="A" x="205.74" y="215.9" smashed="yes" rot="R270">
+<instance part="S4" gate="A" x="205.74" y="215.9" smashed="yes" rot="R270">
 <attribute name="NAME" x="211.455" y="222.25" size="1.778" layer="95" rot="R270"/>
 <attribute name="VALUE" x="198.12" y="222.25" size="1.778" layer="96" rot="R270"/>
 </instance>
-<instance part="SERVO5" gate="A" x="228.6" y="215.9" smashed="yes" rot="R270">
+<instance part="S5" gate="A" x="228.6" y="215.9" smashed="yes" rot="R270">
 <attribute name="NAME" x="234.315" y="222.25" size="1.778" layer="95" rot="R270"/>
 <attribute name="VALUE" x="220.98" y="222.25" size="1.778" layer="96" rot="R270"/>
@@
 <instance part="C15" gate="G$1" x="60.96" y="68.58" smashed="yes" rot="R90"/>
 <instance part="AGND20" gate="VR1" x="38.1" y="116.84" smashed="yes" rot="R180"/>
-<instance part="L2" gate="G$1" x="48.26" y="104.14" smashed="yes" rot="R90">
-<attribute name="NAME" x="53.34" y="102.87" size="1.778" layer="95" rot="R180"/>
+<instance part="L2" gate="G$1" x="45.72" y="101.6" smashed="yes">
+<attribute name="NAME" x="46.99" y="101.6" size="1.778" layer="95" rot="R180"/>
 </instance>
 <instance part="C16" gate="G$1" x="60.96" y="63.5" smashed="yes" rot="R90"/>
@@
 <wire x1="182.88" y1="218.44" x2="182.88" y2="200.66" width="0.1524" layer="91"/>
 <label x="182.88" y="200.66" size="1.778" layer="95" rot="R180" xref="yes"/>
-<pinref part="SERVO3" gate="A" pin="2"/>
+<pinref part="S3" gate="A" pin="2"/>
 </segment>
 <segment>
 <wire x1="144.78" y1="218.44" x2="144.78" y2="200.66" width="0.1524" layer="91"/>
 <label x="144.78" y="200.66" size="1.778" layer="95" rot="R180" xref="yes"/>
-<pinref part="SERVO1" gate="A" pin="2"/>
+<pinref part="S1" gate="A" pin="2"/>
 </segment>
 <segment>
@@
 </segment>
 <segment>
-<pinref part="SERVO2" gate="A" pin="2"/>
+<pinref part="S2" gate="A" pin="2"/>
 <wire x1="162.56" y1="218.44" x2="162.56" y2="203.2" width="0.1524" layer="91"/>
 <label x="152.4" y="203.2" size="1.778" layer="95"/>
 </segment>
 <segment>
-<pinref part="SERVO4" gate="A" pin="2"/>
+<pinref part="S4" gate="A" pin="2"/>
 <wire x1="205.74" y1="218.44" x2="205.74" y2="200.66" width="0.1524" layer="91"/>
 <label x="195.58" y="200.66" size="1.778" layer="95"/>
 </segment>
 <segment>
-<pinref part="SERVO5" gate="A" pin="2"/>
+<pinref part="S5" gate="A" pin="2"/>
 <wire x1="228.6" y1="218.44" x2="228.6" y2="200.66" width="0.1524" layer="91"/>
 <label x="218.44" y="200.66" size="1.778" layer="95"/>
@@
 </segment>
 <segment>
-<pinref part="SERVO1" gate="A" pin="3"/>
+<pinref part="S1" gate="A" pin="3"/>
 <wire x1="142.24" y1="218.44" x2="142.24" y2="213.36" width="0.1524" layer="91"/>
 <pinref part="AGND6" gate="VR1" pin="AGND"/>
@@
 <segment>
 <pinref part="AGND8" gate="VR1" pin="AGND"/>
-<pinref part="SERVO2" gate="A" pin="3"/>
+<pinref part="S2" gate="A" pin="3"/>
 <wire x1="160.02" y1="213.36" x2="160.02" y2="218.44" width="0.1524" layer="91"/>
 </segment>
 <segment>
 <pinref part="AGND9" gate="VR1" pin="AGND"/>
-<pinref part="SERVO3" gate="A" pin="3"/>
+<pinref part="S3" gate="A" pin="3"/>
 <wire x1="180.34" y1="213.36" x2="180.34" y2="218.44" width="0.1524" layer="91"/>
 </segment>
 <segment>
 <pinref part="AGND10" gate="VR1" pin="AGND"/>
-<pinref part="SERVO4" gate="A" pin="3"/>
+<pinref part="S4" gate="A" pin="3"/>
 <wire x1="203.2" y1="213.36" x2="203.2" y2="218.44" width="0.1524" layer="91"/>
 </segment>
 <segment>
 <pinref part="AGND11" gate="VR1" pin="AGND"/>
-<pinref part="SERVO5" gate="A" pin="3"/>
+<pinref part="S5" gate="A" pin="3"/>
 <wire x1="226.06" y1="213.36" x2="226.06" y2="218.44" width="0.1524" layer="91"/>
 </segment>
@@
 <net name="SIGNAL1" class="0">
 <segment>
-<pinref part="SERVO1" gate="A" pin="1"/>
+<pinref part="S1" gate="A" pin="1"/>
 <wire x1="147.32" y1="218.44" x2="147.32" y2="195.58" width="0.1524" layer="91"/>
 <label x="147.32" y="195.58" size="1.778" layer="95" rot="R180" xref="yes"/>
@@
 <net name="SIGNAL2" class="0">
 <segment>
-<pinref part="SERVO2" gate="A" pin="1"/>
+<pinref part="S2" gate="A" pin="1"/>
 <wire x1="165.1" y1="218.44" x2="165.1" y2="195.58" width="0.1524" layer="91"/>
 <label x="165.1" y="195.58" size="1.778" layer="95" rot="R180" xref="yes"/>
@@
 <wire x1="185.42" y1="218.44" x2="185.42" y2="195.58" width="0.1524" layer="91"/>
 <label x="185.42" y="195.58" size="1.778" layer="95" rot="R180" xref="yes"/>
-<pinref part="SERVO3" gate="A" pin="1"/>
+<pinref part="S3" gate="A" pin="1"/>
 </segment>
 <segment>
@@
 <wire x1="208.28" y1="218.44" x2="208.28" y2="195.58" width="0.1524" layer="91"/>
 <label x="208.28" y="195.58" size="1.778" layer="95" rot="R180" xref="yes"/>
-<pinref part="SERVO4" gate="A" pin="1"/>
+<pinref part="S4" gate="A" pin="1"/>
 </segment>
 <segment>
@@
 <wire x1="231.14" y1="218.44" x2="231.14" y2="195.58" width="0.1524" layer="91"/>
 <label x="231.14" y="195.58" size="1.778" layer="95" rot="R180" xref="yes"/>
-<pinref part="SERVO5" gate="A" pin="1"/>
+<pinref part="S5" gate="A" pin="1"/>
 </segment>
 <segment>
@@
 <pinref part="L2" gate="G$1" pin="2"/>
 <wire x1="55.88" y1="68.58" x2="58.42" y2="68.58" width="0.1524" layer="91"/>
-<wire x1="55.88" y1="104.14" x2="55.88" y2="68.58" width="0.1524" layer="91"/>
+<wire x1="66.04" y1="101.6" x2="55.88" y2="68.58" width="0.1524" layer="91"/>
 <junction x="55.88" y="68.58"/>
 </segment>
@@
 <wire x1="40.64" y1="88.9" x2="40.64" y2="101.6" width="0.1524" layer="91"/>
 <pinref part="L2" gate="G$1" pin="1"/>
-<wire x1="40.64" y1="101.6" x2="40.64" y2="104.14" width="0.1524" layer="91"/>
-<wire x1="40.64" y1="101.6" x2="38.1" y2="101.6" width="0.1524" layer="91"/>
+<wire x1="40.64" y1="101.6" x2="45.72" y2="101.6" width="0.1524" layer="91"/>
 <junction x="40.64" y="101.6"/>
-<wire x1="38.1" y1="101.6" x2="38.1" y2="104.14" width="0.1524" layer="91"/>
+<wire x1="40.64" y1="101.6" x2="38.1" y2="104.14" width="0.1524" layer="91"/>
 <pinref part="C18" gate="G$1" pin="1"/>
 </segment>
