File: ProstheticsEagle/circuitdraft.sch (EAGLE design)
At the start: 49 parts, among them IC1 BQ25887RGER, IC2 TPS54627DDAR, Q1 16 MHz

Commit message: aa
Parts:
- C11, C12: value 22 pF -> 22 uF
- C4, C5: value 10 pF -> 10 uF
- C6: value .1 pF -> .1 uF
Changed lines of the file:
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@@
 <part name="C3" library="rcl" library_urn="urn:adsk.eagle:library:334" deviceset="C-US" device="C0805" package3d_urn="urn:adsk.eagle:package:23617/2" value="22 pF"/>
 <part name="AGND5" library="supply1" library_urn="urn:adsk.eagle:library:371" deviceset="AGND" device=""/>
-<part name="C4" library="rcl" library_urn="urn:adsk.eagle:library:334" deviceset="C-US" device="C0805" package3d_urn="urn:adsk.eagle:package:23617/2" value="10 pF"/>
-<part name="C5" library="rcl" library_urn="urn:adsk.eagle:library:334" deviceset="C-US" device="C0805" package3d_urn="urn:adsk.eagle:package:23617/2" value="10 pF"/>
-<part name="C6" library="rcl" library_urn="urn:adsk.eagle:library:334" deviceset="C-US" device="C0805" package3d_urn="urn:adsk.eagle:package:23617/2" value=".1 pF"/>
+<part name="C4" library="rcl" library_urn="urn:adsk.eagle:library:334" deviceset="C-US" device="C0805" package3d_urn="urn:adsk.eagle:package:23617/2" value="10 uF"/>
+<part name="C5" library="rcl" library_urn="urn:adsk.eagle:library:334" deviceset="C-US" device="C0805" package3d_urn="urn:adsk.eagle:package:23617/2" value="10 uF"/>
+<part name="C6" library="rcl" library_urn="urn:adsk.eagle:library:334" deviceset="C-US" device="C0805" package3d_urn="urn:adsk.eagle:package:23617/2" value=".1 uF"/>
 <part name="AGND12" library="supply1" library_urn="urn:adsk.eagle:library:371" deviceset="AGND" device=""/>
 <part name="R3" library="rcl" library_urn="urn:adsk.eagle:library:334" deviceset="R-US_" device="R0603" package3d_urn="urn:adsk.eagle:package:23555/3" value="10000 Ohms"/>
@@
 <part name="C10" library="rcl" library_urn="urn:adsk.eagle:library:334" deviceset="C-US" device="C0805" package3d_urn="urn:adsk.eagle:package:23617/2" value="0.1 uF"/>
 <part name="L1" library="SamacSys_Parts" deviceset="RLB0912-3R3ML" device=""/>
-<part name="C11" library="rcl" library_urn="urn:adsk.eagle:library:334" deviceset="C-US" device="C0805" package3d_urn="urn:adsk.eagle:package:23617/2" value="22 pF"/>
-<part name="C12" library="rcl" library_urn="urn:adsk.eagle:library:334" deviceset="C-US" device="C0805" package3d_urn="urn:adsk.eagle:package:23617/2" value="22 pF"/>
+<part name="C11" library="rcl" library_urn="urn:adsk.eagle:library:334" deviceset="C-US" device="C0805" package3d_urn="urn:adsk.eagle:package:23617/2" value="22 uF"/>
+<part name="C12" library="rcl" library_urn="urn:adsk.eagle:library:334" deviceset="C-US" device="C0805" package3d_urn="urn:adsk.eagle:package:23617/2" value="22 uF"/>
 <part name="AGND14" library="supply1" library_urn="urn:adsk.eagle:library:371" deviceset="AGND" device=""/>
 <part name="AGND15" library="supply1" library_urn="urn:adsk.eagle:library:371" deviceset="AGND" device=""/>
@@
 </instance>
 <instance part="C4" gate="G$1" x="182.88" y="68.58" smashed="yes" rot="R180">
-<attribute name="NAME" x="185.039" y="65.024" size="1.778" layer="95" rot="R90"/>
-<attribute name="VALUE" x="179.959" y="65.024" size="1.778" layer="96" rot="R90"/>
+<attribute name="NAME" x="178.816" y="68.199" size="1.778" layer="95" rot="R180"/>
+<attribute name="VALUE" x="181.356" y="65.659" size="1.778" layer="96" rot="R180"/>
 </instance>
 <instance part="C5" gate="G$1" x="193.04" y="68.58" smashed="yes" rot="R180">
-<attribute name="NAME" x="195.199" y="65.024" size="1.778" layer="95" rot="R90"/>
-<attribute name="VALUE" x="190.119" y="65.024" size="1.778" layer="96" rot="R90"/>
+<attribute name="NAME" x="196.596" y="65.659" size="1.778" layer="95" rot="R180"/>
+<attribute name="VALUE" x="191.516" y="65.659" size="1.778" layer="96" rot="R180"/>
 </instance>
 <instance part="C6" gate="G$1" x="205.74" y="68.58" smashed="yes" rot="R180">
-<attribute name="NAME" x="207.899" y="65.024" size="1.778" layer="95" rot="R90"/>
-<attribute name="VALUE" x="202.819" y="65.024" size="1.778" layer="96" rot="R90"/>
+<attribute name="NAME" x="209.296" y="65.659" size="1.778" layer="95" rot="R180"/>
+<attribute name="VALUE" x="204.216" y="65.659" size="1.778" layer="96" rot="R180"/>
 </instance>
 <instance part="AGND12" gate="VR1" x="210.82" y="63.5" smashed="yes">
-<attribute name="VALUE" x="208.28" y="58.42" size="1.778" layer="96" rot="R90"/>
+<attribute name="VALUE" x="218.44" y="66.04" size="1.778" layer="96" rot="R180"/>
 </instance>
 <instance part="R3" gate="G$1" x="177.8" y="50.8" smashed="yes">
@@
 </instance>
 <instance part="C8" gate="G$1" x="182.88" y="38.1" smashed="yes">
-<attribute name="NAME" x="180.721" y="41.656" size="1.778" layer="95" rot="R180"/>
+<attribute name="NAME" x="188.341" y="31.496" size="1.778" layer="95" rot="R180"/>
 <attribute name="VALUE" x="185.801" y="41.656" size="1.778" layer="96" rot="R270"/>
 </instance>
@@
 </instance>
 <instance part="C10" gate="G$1" x="228.6" y="48.26" smashed="yes" rot="R270">
-<attribute name="NAME" x="232.156" y="50.419" size="1.778" layer="95" rot="R180"/>
+<attribute name="NAME" x="234.696" y="50.419" size="1.778" layer="95" rot="R180"/>
 <attribute name="VALUE" x="232.156" y="45.339" size="1.778" layer="96" rot="R180"/>
 </instance>

Commit message: added new inductor
Parts:
- L1: value RLB0912-3R3ML -> IHLP2020CZER3R3M01; device SamacSys_Parts:RLB0912-3R3ML -> ind2:IHLP2020CZER3R3M01
- Q1: device crystal:CRYSTALHC49S -> crystal-geyer_V1_0:KX-5
- renumbered C10 to C1.7, C11 to C1.8, C12 to C1.9, C4 to C1.1, C5 to C1.2, C6 to C1.3, C7 to C1.4, C8 to C1.6, C9 to C1.5, R3 to R1.3, R4 to R1.1, R5 to R1.2
Connections:
- net N$14: now also L1.2; no longer L1.1
- net POWER: now also L1.1; no longer L1.2

Commit message: Reorganized alot of things. Created different grounds
Parts:
- added BU: (no value), pinhead:PINHD-1X2
- renumbered C13 to C2.3, C14 to C2.2, C15 to C2.5, C16 to C2.4, C17 to C2.1, C18 to C2.6, R10 to R2.1, R11 to R2.4, R12 to R2.9, R13 to R2.8, R14 to R2.6, R6 to R2.7, R7 to R2.3, R8 to R2.2, R9 to R2.5
Connections:
- new net GND: BATIO.3, C1.1.1, C1.2, C1.2.1, C1.3.1, C1.5.2, C1.8.2, C1.9.2, C2.1, C2.1.1, C2.2.2, C2.3.1, C2.4.2, C2.6.2, C3.1, IC1.GND_2, IC1.ILIM, IC2.EP, IC2.GND, ISP.6, LED.2, MYO.2, R2.9.1, S1.3, S2.3, S3.3, S4.3, S5.3, TS.2, U$1.GND2
- new net INTERRUPT?: U$1.(RXD1/INT2)PD2
- net AGND: no longer BATIO.3, C1.1.1, C1.2, C1.2.1, C1.3.1, C1.5.2, C1.8.2, C1.9.2, C2.1, C2.1.1, C2.2.2, C2.3.1, C2.4.2, C2.6.2, C3.1, IC1.GND_2, IC1.ILIM, IC2.EP, IC2.GND, ISP.6, LED.2, MYO.2, R2.9.1, S1.3, S2.3, S3.3, S4.3, S5.3, TS.2, U$1.GND2
Other:
- moved on the sheet: C3

Commit message: Ahmad's changes
Parts:
- C1.5, C1.6: device rcl:C-USC0805 -> rcl:C-USC0603
Connections:
- removed net AGND: C1.6.2, R1.2.2
- net GND: now also C1.6.2, R1.2.2
Changed lines of the file:
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@@
 <part name="C1.4" library="rcl" library_urn="urn:adsk.eagle:library:334" deviceset="C-US" device="C0805" package3d_urn="urn:adsk.eagle:package:23617/2" value="10 pF"/>
 <part name="R1.2" library="rcl" library_urn="urn:adsk.eagle:library:334" deviceset="R-US_" device="R0603" package3d_urn="urn:adsk.eagle:package:23555/3" value="22100 Ohms"/>
-<part name="C1.6" library="rcl" library_urn="urn:adsk.eagle:library:334" deviceset="C-US" device="C0805" package3d_urn="urn:adsk.eagle:package:23617/2" value="8200 pF"/>
-<part name="C1.5" library="rcl" library_urn="urn:adsk.eagle:library:334" deviceset="C-US" device="C0805" package3d_urn="urn:adsk.eagle:package:23617/2" value="1 uF"/>
+<part name="C1.6" library="rcl" library_urn="urn:adsk.eagle:library:334" deviceset="C-US" device="C0603" package3d_urn="urn:adsk.eagle:package:23616/2" value="8200 pF"/>
+<part name="C1.5" library="rcl" library_urn="urn:adsk.eagle:library:334" deviceset="C-US" device="C0603" package3d_urn="urn:adsk.eagle:package:23616/2" value="1 uF"/>
 <part name="C1.7" library="rcl" library_urn="urn:adsk.eagle:library:334" deviceset="C-US" device="C0805" package3d_urn="urn:adsk.eagle:package:23617/2" value="0.1 uF"/>
 <part name="L1" library="ind2" deviceset="IHLP2020CZER3R3M01" device=""/>
 <part name="C1.8" library="rcl" library_urn="urn:adsk.eagle:library:334" deviceset="C-US" device="C0805" package3d_urn="urn:adsk.eagle:package:23617/2" value="22 uF"/>
 <part name="C1.9" library="rcl" library_urn="urn:adsk.eagle:library:334" deviceset="C-US" device="C0805" package3d_urn="urn:adsk.eagle:package:23617/2" value="22 uF"/>
-<part name="AGND14" library="supply1" library_urn="urn:adsk.eagle:library:371" deviceset="AGND" device=""/>
 <part name="AGND15" library="supply1" library_urn="urn:adsk.eagle:library:371" deviceset="GND" device=""/>
 <part name="IC1" library="SamacSys_Parts" deviceset="BQ25887RGER" device=""/>
@@
 <part name="AGND13" library="supply1" library_urn="urn:adsk.eagle:library:371" deviceset="GND" device=""/>
 <part name="LED" library="pinhead" library_urn="urn:adsk.eagle:library:325" deviceset="PINHD-1X3" device="" package3d_urn="urn:adsk.eagle:package:22458/2"/>
-<part name="AGND16" library="supply1" library_urn="urn:adsk.eagle:library:371" deviceset="AGND" device=""/>
 <part name="BU" library="pinhead" library_urn="urn:adsk.eagle:library:325" deviceset="PINHD-1X2" device="" package3d_urn="urn:adsk.eagle:package:22435/2"/>
 </parts>
@@
 <attribute name="VALUE" x="277.241" y="39.116" size="1.778" layer="96" rot="R180"/>
 </instance>
-<instance part="AGND14" gate="VR1" x="182.88" y="25.4" smashed="yes">
-<attribute name="VALUE" x="180.34" y="20.32" size="1.778" layer="96"/>
-</instance>
 <instance part="AGND15" gate="1" x="172.72" y="27.94" smashed="yes">
 <attribute name="VALUE" x="170.18" y="22.86" size="1.778" layer="96"/>
@@
 <attribute name="NAME" x="270.51" y="117.475" size="1.778" layer="95"/>
 <attribute name="VALUE" x="270.51" y="104.14" size="1.778" layer="96"/>
-</instance>
-<instance part="AGND16" gate="VR1" x="160.02" y="25.4" smashed="yes">
-<attribute name="VALUE" x="157.48" y="20.32" size="1.778" layer="96"/>
 </instance>
 <instance part="BU" gate="G$1" x="254" y="139.7" smashed="yes">
@@
 <pinref part="C1.5" gate="G$1" pin="2"/>
 <pinref part="AGND15" gate="1" pin="GND"/>
-<wire x1="172.72" y1="33.02" x2="172.72" y2="30.48" width="0.1524" layer="91"/>
+<wire x1="172.72" y1="30.48" x2="172.72" y2="33.02" width="0.1524" layer="91"/>
+<pinref part="R1.2" gate="G$1" pin="2"/>
+<wire x1="160.02" y1="27.94" x2="160.02" y2="20.32" width="0.1524" layer="91"/>
+<wire x1="160.02" y1="20.32" x2="182.88" y2="20.32" width="0.1524" layer="91"/>
+<pinref part="C1.6" gate="G$1" pin="2"/>
+<wire x1="182.88" y1="20.32" x2="182.88" y2="30.48" width="0.1524" layer="91"/>
+<label x="182.88" y="20.32" size="1.778" layer="95"/>
+<wire x1="182.88" y1="30.48" x2="182.88" y2="33.02" width="0.1524" layer="91"/>
+<wire x1="172.72" y1="30.48" x2="182.88" y2="30.48" width="0.1524" layer="91"/>
+<junction x="172.72" y="30.48"/>
+<junction x="182.88" y="30.48"/>
 </segment>
 <segment>
@@
 </segment>
 </net>
-<net name="AGND" class="0">
-<segment>
-<pinref part="AGND14" gate="VR1" pin="AGND"/>
-<wire x1="182.88" y1="33.02" x2="182.88" y2="27.94" width="0.1524" layer="91"/>
-<pinref part="C1.6" gate="G$1" pin="2"/>
-</segment>
-<segment>
-<pinref part="R1.2" gate="G$1" pin="2"/>
-<pinref part="AGND16" gate="VR1" pin="AGND"/>
-</segment>
-</net>
